File: KiCAD/CPU/CPU.kicad_sch (KiCad schematic)
At the start: 60 parts, among them J1 Address, J2 Data, J3 RDN, J4 WRN, U12 74LS139, U16 PhaseGenerator, U21 74HC86, U27 74HC86, U28 Small_OR3, U3 74LS125, U4 74LCX07, U5 74LS125, U6 74LCX07, U7 74LCX07

Commit message: Simplified ALU and register file data paths
Parts:
- removed +, +1: +, symbol UKMaker:Generic_Adder
- removed ALU1: ~, symbol UKMaker:Generic_ALU
- removed MUX13, MUX16, MUX19: MUX4, symbol UKMaker:Generic_MUX4
- removed MUX14: MUX3, symbol UKMaker:Generic_MUX3
- removed MUX15, MUX17, MUX18: MUX2, symbol UKMaker:Generic_MUX2
- removed MUX8_R1: ~, symbol UKMaker:Generic_MUX8_R
- removed U1: ~, symbol UKMaker:Generic_DualPortRegisterFile
- removed U15, U8, U9: ~, symbol UKMaker:Generic_REGISTER
- removed U18: ~, symbol UKMaker:Generic_Small_INV
- removed U22: ~, symbol UKMaker:Generic_Small_OR2
- removed U23: ~, symbol UKMaker:Generic_Register_With_Enable
- removed U24, U25, U26: ~, symbol UKMaker:Generic_Small_AND2
- removed U27: 74HC86, symbol 74xx:74HC86
- added MUX13: MUX3, symbol UKMaker:Generic_MUX3
- added MUX14, MUX20: MUX2, symbol UKMaker:Generic_MUX2
- added U1: ~, symbol UKMaker:Generic_DualPortRegisterFile_ByteEnable
Connections:
- net ALUA_PP is gone; now on net ALUB_CONSTX: MUX11. (SEL)
- net REGA_DINX is gone; now on net ALUB_CONSTX: MUX11. (SEL)
- net 0: now also MUX11. (SEL); no longer MUX8_R2. (SEL)
- net 1: now also MUX11. (SEL)
- net 2: now also MUX11. (SEL)
- net ABUS_X: now also MUX13. (SEL)
- net ALUA_DATA: now also MUX13. (SEL)
- net ALUB_DATA: now also MUX14. (SEL), U1. (WEN)
- net ALU_R: now also ALU2. (R), MUX13. (SEL), MUX14. (SEL), U1. (WEN); no longer MUX11. (SEL)
- net ARGA_X: no longer MUX6. (SEL)
- net DBUS_X: now also MUX14. (SEL)
- net DIN: now also MUX20. (SEL)
- net PC_A: now also MUX13. (SEL), MUX20. (SEL); no longer MUX11. (SEL)
- net REGA_DOUT: now also U1. (WEN)
- net REGA_EN: now also U1. (WEN)
- net REGA_WEN: now also U1. (WEN)
- net REGB_EN: now also U1. (WEN)
- net REGB_WEN: now also U1. (WEN)
- net RL: now also MUX6. (SEL)
- net at +. (R): now also U2. (LD); no longer MUX12. (SEL)
- net at U3.2: now also MUX14. (SEL)
- net ALUB_CONSTX: now reaches MUX11. (SEL)
- net at U5.2: now also MUX13. (SEL)
- new net: MUX6. (SEL), U1. (WEN)
- new net: ALU2. (R), U17. (LD)
- new net: U13. (Q), U14. (Q), U20. (Q), U29. (Q)
- new net: MUX6_R2. (SEL), MUX9. (SEL)
- new net: MUX9. (SEL), U1. (WEN)
- new net: +. (R), MUX12. (SEL)
- new net: U20. (Q), U28. (Q)
- new net: +. (R), MUX10. (SEL)
- new net: U13. (Q), U19. (Q)
- new net: MUX11. (SEL), MUX8_R2. (SEL)
- new net: MUX20. (SEL), U1. (WEN)
- new net REGA_BYTE_ENX: U1. (WEN)
- new net REGB_BYTE_ENX: U1. (WEN)
- new net REGB_DINX: MUX20. (SEL)
Other:
- moved on the sheet: MUX6, MUX6_R2, MUX9, U17

Commit message: Updated for branch decoding and interrupts
Parts:
- removed MUX10, MUX11, MUX6: MUX3, symbol UKMaker:Generic_MUX3
- removed MUX12, MUX14, MUX5, MUX9: MUX2, symbol UKMaker:Generic_MUX2
- removed MUX6_R2: MUX6_R, symbol UKMaker:Generic_MUX6_R
- removed MUX8_R2: ~, symbol UKMaker:Generic_MUX8_R
- removed U10: ~, symbol UKMaker:Generic_REGISTER
- removed U12: 74LS139, symbol 74xx:74LS139
- removed U14: ~, symbol UKMaker:Generic_Small_AND2
- removed U19: ~, symbol UKMaker:Generic_Small_INV
- removed U2: ~, symbol UKMaker:Generic_Register_With_Enable
- removed U28: Small_OR3, symbol UKMaker:Generic_Small_OR3
- added J5: WR1N, symbol Connector_Generic:Conn_01x01
- added MUX11: MUX4, symbol UKMaker:Generic_MUX4
- added MUX14: MUX3, symbol UKMaker:Generic_MUX3
- added MUX16: MUX2, symbol UKMaker:Generic_MUX2
- added MUX17, MUX18: MUX6, symbol UKMaker:Generic_MUX6
- added MUX19, MUX6, MUX9: ~, symbol UKMaker:Generic_MUX5
- added MUX4_R1: ~, symbol UKMaker:Generic_MUX4_R
- added MUX5: ~, symbol UKMaker:Generic_MUX7
- added MUX8_R1: ~, symbol UKMaker:Generic_MUX8_R
- added U10, U12: ~, symbol UKMaker:Generic_Small_OR2
- added U30: 74LCX07, symbol 74xx:74LCX07
- added U33, U34, U35: ~, symbol UKMaker:Generic_Register_With_Enable
- J4: value WRN -> WR0N
- MUX2: value MUX3 -> ~
- MUX3: value MUX4 -> ~
- MUX4: value MUX5 -> ~
Connections:
- net PC_BASEX_0 is gone; now on net PC_BASEX: U13. (Q)
- net REGB_DINX is gone; now on net PC_BASEX: MUX20. (SEL)
- net RET_X is gone; now on net PC_BASEX: U13. (Q)
- net 0: now also MUX20. (SEL), MUX18. (SEL)
- net 1: now also MUX18. (SEL)
- net 2: now also MUX16. (SEL), MUX18. (SEL)
- net ALUA_DATA: now also MUX14. (SEL), MUX18. (SEL); no longer MUX13. (SEL)
- net ALUA_SRCX: now also MUX18. (SEL)
- net ALUB_DATA: now also MUX9. (SEL); no longer U1. (WEN)
- net ALUB_SRCX: now also MUX9. (SEL)
- net ALU_R: now also MUX14. (SEL), MUX4_R1. (SEL)
- net ARGA_X: now also MUX11. (SEL)
- net ARGB_X: now also MUX6. (SEL)
- net DBUS_X: now also MUX14. (SEL)
- net DIN: now also MUX4_R1. (SEL); no longer MUX20. (SEL)
- net FETCH: now also U33. (LD), U34. (LD), U35. (LD)
- net FP: now also MUX6. (SEL)
- net PC_A: now also U33. (LD)
- net PC_OFFSETX: now also MUX16. (SEL)
- net RA: now also MUX11. (SEL)
- net RB: now also MUX11. (SEL), MUX6. (SEL)
- net REGA_ADDRX: now also MUX11. (SEL)
- net REGB_ADDRX: now also MUX6. (SEL)
- net RL: now also MUX11. (SEL)
- net RS: now also MUX6. (SEL)
- net SP: now also MUX6. (SEL)
- net U4: now also MUX9. (SEL)
- net U4.0: now also MUX9. (SEL)
- net U6: now also MUX18. (SEL)
- net U6.0: now also MUX18. (SEL)
- net U8: now also MUX9. (SEL)
- net U8H: now also MUX9. (SEL)
- net WRN: now also U10. (Q), U12. (Q); no longer U7.1
- net at U3.2: now also MUX14. (SEL)
- net PC_A_NEXT: now reaches +. (R)
- net PC_A_NEXT: now also MUX19. (SEL), MUX4_R1. (SEL), U34. (LD), U35. (LD)
- new net: MUX6. (SEL), U1. (WEN)
- new net: ALU2. (R), U17. (LD)
- new net: +. (R), MUX20. (SEL)
- new net: U13. (Q), U20. (Q), U29. (Q)
- new net: U12. (Q), U30.1
- new net: MUX19. (SEL), U33. (LD)
- new net: +. (R), MUX16. (SEL)
- new net: U10. (Q), U7.1
- new net: J5.1 (Pin_1), U30.2
- new net: MUX11. (SEL), U1. (WEN)
- new net: MUX4_R1. (SEL), U1. (WEN)
- new net ALUA_DATAH: MUX14. (SEL)
- new net ALUA_DIN: MUX18. (SEL)
- new net ALUB_DIN: MUX13. (SEL)
- new net DOUT_BYTE_ENX: U10. (Q), U12. (Q)
- new net INTR0: MUX19. (SEL), U35. (LD)
- new net INTR1: MUX19. (SEL), U34. (LD)
- new net INTV0: MUX19. (SEL)
- new net INTV1: MUX19. (SEL)
- new net JMPX: U13. (Q), U20. (Q)
- new net JRX: U13. (Q)
- new net PC_D: MUX16. (SEL)
- new net PC_ENX: U33. (LD)
- new net PC_LD_INT0X: U35. (LD)
- new net PC_LD_INT1X: U34. (LD)
- new net PC_NEXTX: MUX19. (SEL)
- new net REGA_DINX: MUX4_R1. (SEL)
- new net REGB_DOUT: MUX9. (SEL), U1. (WEN)
Other:
- added sheet Data Flows (DataFlows.kicad_sch)
- note added: "DINH"
- note added: "Decode Logic"
- note removed: "ARGF REGA_ADDRX REGB_ADDRX ALUA_SRCX ALUB_SRCX WR_A WR_B RD_A RD_B ------------------------------------------------------------------------------------------------------- 0 0 - Ra,Rb 0 0 - ARGA_X 0 0 - ARGB_X 0 - REGA 0 0 0 - REGB 1 0 1 1 0 1 - Ra,U4 0 0 - ARGA_X 0 0 - ARGA_X 0 - REGA 0 1 0 - U4 1 0 1 0 1 0 - RB,U8L 1 0 - RB 0 0 - ARGA_X 0 - REGA 1 0 0 - U8L 1 0 1 0 1 1 - RA,U8H.RBL 0 1 - RB 0 0 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"
- note removed: "Decoding logic"
- note removed: "JP U8H.RBL - CC_APPLYX = 0 - PC_BASEX = 0 - PC_OFFSETX = PC_D - PC_EN = 1 - JMP_X = 1 - REGB_ADDRX = RB - REGB_EN = 1"
- note removed: "JR Rb - CC_APPLYX = 0 - PC_BASEX = PC - PC_OFFSETX = PC_D - PC_EN = 1 - JMP_X = 1 - REGB_ADDRX = ARGB_X - REGB_EN = 1"
- note removed: "LD Ra,(Rb) - REGA_ADDRX = ARGA_X - WRA_EN = 1 - REGA_DINX = DIN - ALUA_SRCX = 0 (IGN) - ALU_OPX = MOV (IGN) - REGB_ADDRX = ARGB_X - RDB_EN = 1 - ABUS_X = REGB - MEM_READ = 1 LD Ra,(Rb++) - REGA_ADDRX = ARGA_X - WRA_EN = 1 - REGA_DINX = DIN - ALUA_SRCX = 2 (1 for Byte ops) - ALU_OPX = PLUS - REGB_ADDRX = ARGB_X - RDB_EN = 1 - WRB_EN = 1 - REGB_DINX = ALU_R - ABUS_X = REGB - MEM_READ = 1 LD Ra,(--R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"
- note removed: "MODEF INCF LDSF ----------------------------------------- 0 0 - Rb,(Ra) 0 0 - IGN 0 0 - LD 0 1 - Rb,(FP+U4) 0 1 - IGN 0 1 - LD_B 1 0 - Rb,(SP+U4) 1 0 - X++ 1 0 - ST 1 1 - Rb,(RS+U4) 1 1 - --X 1 1 - ST_B"
- note removed: "SKIPF JPF CCF -------------------------------------------- 0 0 - Always 0 0 - JP Rb 0 0 - CCC 0 1 - Always 0 1 - JP U8H.RBL 0 1 - CCZ 1 0 - CC Match 1 0 - JR Rb 1 0 - CCP 1 1 - CC !Match 1 1 - JR U8H.RBL 1 1 - CCM JP Rb - CC_APPLYX = 0 - PC_BASEX = 0 - PC_OFFSETX = PC_D - PC_EN = 1 - JMP_X = 1 - REGB_ADDRX = ARGB_X - REGB_EN = 1 - REGA_ADDRX = RL - REGA_WEN = 1 - REGA_DINX = PC_A"
- note removed: "ST (FP++ +U4),Ra ------------------ ALUB_SRCX = U4 ALUA_SRCX = ALUA_PP REGA_ADDRX = FP REGB_ADDRX = ARGBX ABYS_X = ALU_R DBUS_X = REGA_DOUT"
- note removed: "[11:10]"
- note removed: "[13:10]"
- note removed: "[13:12]"
- note removed: "[15:14]"
- note removed: "[3:0]"
- note removed: "[3:0].0"
- note removed: "[7:0]"
- note removed: "[7:4]"
- note removed: "[9:8]"
- moved on the sheet: ALU2, J1, J2, J3, J4, MUX1, MUX13, MUX2, MUX3, MUX4, U1, U16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

Commit message: Started design of debugV2 with snooping
Parts:
- removed J1: Address, symbol Connector_Generic:Conn_01x01
- removed J2: Data, symbol Connector_Generic:Conn_01x01
- removed J3: RDN, symbol Connector_Generic:Conn_01x01
- removed J4: WR0N, symbol Connector_Generic:Conn_01x01
- removed J5: WR1N, symbol Connector_Generic:Conn_01x01
- removed MUX13, MUX14: MUX3, symbol UKMaker:Generic_MUX3
- removed MUX16, MUX20: MUX2, symbol UKMaker:Generic_MUX2
- removed MUX18: MUX6, symbol UKMaker:Generic_MUX6
- removed MUX4_R1: ~, symbol UKMaker:Generic_MUX4_R
- removed MUX9: ~, symbol UKMaker:Generic_MUX5
- removed U10, U12: ~, symbol UKMaker:Generic_Small_OR2
- removed U17: ~, symbol UKMaker:Generic_REGISTER
- removed U3, U5: 74LS125, symbol 74xx:74LS125
- removed U30, U4, U6, U7: 74LCX07, symbol 74xx:74LCX07
- added +1: +, symbol UKMaker:Generic_Adder
- added J? (x5): Conn_01x01, symbol Connector_Generic:Conn_01x01
- added MUX10 (x2): MUX2, symbol UKMaker:Generic_MUX2
- added MUX3, MUX? (x2): MUX4, symbol UKMaker:Generic_MUX4
- added MUX?: MUX5, symbol UKMaker:Generic_MUX5
- added MUX? (x2): MUX3, symbol UKMaker:Generic_MUX3
- added MUX? (x2): ~, symbol UKMaker:Generic_MUX8
- added U14 (x2), U? (x2): ~, symbol UKMaker:Generic_Small_AND2
- added U36, U? (x5): ~, symbol UKMaker:Generic_Small_INV
- added U? (x4): ~, symbol UKMaker:Generic_Register_With_Enable
- added U? (x5): ~, symbol UKMaker:Generic_Small_TRISTATE_BUF
- added U? (x4): ~, symbol UKMaker:Generic_Latch
- added U?: ~, symbol UKMaker:Generic_REGISTER
- added U?: ~, symbol UKMaker:Generic_Small_BUF
- added U? (x3): ~, symbol UKMaker:Generic_Small_OR2
- MUX?: renamed from MUX6; value ~ -> MUX5
- MUX?: renamed from MUX4; value ~ -> MUX5
- MUX?: renamed from MUX3; value ~ -> MUX4
- MUX?: renamed from MUX19; value ~ -> MUX5
- MUX?: renamed from MUX2; value ~ -> MUX3
- renumbered + to +?, ALU2 to ALU?, MUX8_R1 to MUX8_R?, MUX1 to MUX?, MUX8 to MUX?, MUX5 to MUX?, MUX11 to MUX?, MUX7 to MUX?, MUX17 to MUX?, U35 to U?, U20 to U?, U29 to U?, U33 to U?, U34 to U?, U13 to U?, U21 to U?, U1 to U?, U16 to U?, U11 to U?
Connections:
- net CCM is gone; now on net CC_SELECTX: MUX?. (SEL)
- net CCV is gone; now on net CC_SELECTX: MUX?. (SEL)
- net 0: now also MUX?. (SEL), MUX?. (SEL), MUX?. (SEL), MUX?. (SEL)
- net 1: now also MUX?. (SEL)
- net 2: now also +1. (R), MUX?. (SEL), MUX?. (SEL)
- net ABUS_OEN: now also U?. (Q)
- net ALUA_DATA: now also MUX?. (SEL)
- net ALUA_SRCX: now also MUX?. (SEL)
- net ALUB_DATA: now also MUX?. (SEL), MUX?. (SEL)
- net ALUB_SRCX: now also MUX?. (SEL)
- net ALU_R: now also MUX3. (SEL), MUX?. (SEL), MUX?. (SEL)
- net CCL_LD: now also U?. (LD), U?. (LD), U?. (LD)
- net CCn: now also MUX3. (SEL), MUX?. (SEL)
- net CLK: now also U?. (DOUT), U?. (DOUT), U?. (DOUT), U?. (LD), U?. (LD), U?. (Q)
- net DBUS_OEN: now also U?. (DOUT), U?. (Q)
- net DECODE: now also U?. (LD)
- net DIN: now also MUX?. (SEL), MUX?. (SEL), U?. (LD), U?. (Q)
- net FETCH: now also U?. (LD)
- net JRX: now also U?. (Q); no longer U?. (Q)
- net PC_A: now also MUX?. (SEL), MUX?. (SEL)
- net PC_A_NEXT: now also U?. (LD), +1. (R); no longer +?. (R), U?. (LD), U?. (LD)
- net PC_BASEX: now also MUX?. (SEL)
- net PC_ENX: now also U14. (Q); no longer U?. (LD)
- net PC_OFFSETX: now also MUX?. (SEL)
- net PG_CLR: now also U?. (LD)
- net REGA_DINX: now also MUX?. (SEL)
- net REGA_DOUT: now also MUX3. (SEL), MUX?. (SEL)
- net REGB_DOUT: now also MUX?. (SEL), MUX?. (SEL)
- net RESET: now also U?. (DOUT), U?. (DOUT), U?. (DOUT), U?. (DOUT), U?. (LD), U?. (LD), U?. (LD)
- net U4: now also MUX?. (SEL)
- net U8: now also MUX?. (SEL)
- net U8H: now also MUX?. (SEL)
- net at +?. (R): now also MUX?. (SEL)
- new net: ALU?. (R), U?. (LD), U?. (LD), U?. (LD)
- new net: MUX?. (SEL), U?. (LD) (x3)
- new net: J?.1 (Pin_1), U?. (Q) (x4)
- new net: +1. (R), U?. (LD)
- new net: U14. (Q), U?. (LD), U?. (LD)
- new net: U14. (Q), U36. (Q)
- new net: U?. (DOUT), U?. (Q) (x4)
- new net: MUX?. (SEL), U?. (WEN) (x3)
- new net: U?. (Q), U?. (Q) (x4)
- new net: +?. (R), MUX?. (SEL), U?. (LD), U?. (LD)
- new net: J?.1 (Pin_1), U?. (Q), U?. (Q)
- new net: MUX10. (SEL), MUX?. (SEL)
- new net: U?. (Q), U?. (Q), U?. (Q) (x2)
- new net: U?. (DOUT), U?. (Q), U?. (Q)
- new net: +?. (R), MUX?. (SEL)
- new net -1: MUX?. (SEL)
- new net -2: MUX?. (SEL)
- new net 4: MUX?. (SEL)
- new net ADDR_BUF: MUX?. (SEL), U14. (Q), U?. (Q), U?. (Q), U?. (Q)
- new net ADDR_BUSX: MUX?. (SEL)
- new net AT_BKP: U36. (Q)
- new net BUSEN: U?. (Q), U?. (Q), U?. (Q)
- new net BYTEX: U14. (Q), U?. (Q), U?. (Q)
- new net CCC: MUX?. (SEL)
- new net CCL_EN0X: U?. (LD)
- new net CCL_EN1X: U?. (LD)
- new net CCL_ENRX: U?. (LD)
- new net CCS: MUX?. (SEL)
- new net CC_REGX: MUX?. (SEL)
- new net DATA_BUSX: MUX3. (SEL)
- new net DEBUG_MA: MUX?. (SEL)
- new net DEBUG_MD: MUX3. (SEL)
- new net DINH: MUX10. (SEL)
- new net DINL: MUX10. (SEL)
- new net DOUT_BUF: MUX10. (SEL), U?. (Q)
- new net HERE: MUX?. (SEL), MUX?. (SEL), U?. (LD)
- new net HIGH_BYTEX: MUX10. (SEL), MUX10. (SEL), U14. (Q)
- new net INSTRUCTION: U?. (LD)
- new net RDN_BUF: U?. (DOUT), U?. (Q)
- new net RDX: U?. (Q)
- new net S8: MUX?. (SEL)
- new net U4_0: MUX?. (SEL)
- new net U5: MUX?. (SEL)
- new net U5_0: MUX?. (SEL)
- new net WRN0_BUF: U?. (DOUT), U?. (Q)
- new net WRN1_BUF: U?. (DOUT), U?. (Q)
- new net WRX: U?. (Q), U?. (Q)
- new net {HB,LB}: MUX10. (SEL), MUX3. (SEL)
Other:
- added sheet Debug V2 (debugV2.kicad_sch)
- added sheet DebugBlocks (debugBlocks.kicad_sch)
- added sheet DebugSerialPort (debugSerialPort.kicad_sch)
- added sheet InstructionDecode (instructionDecoder.kicad_sch)
- added sheet MCU (mcu.kicad_sch)
- note removed: "DINH"
- moved on the sheet: ALU?, MUX8_R?, MUX?, U?
